File: Daisy_Amps/Daisy_Amps.kicad_sch (KiCad schematic)
At the start: 5 parts, among them J1 Power and Ground, U5 Daisy_Seed

Commit message: schematic done
Parts:
- Audio_in_jack1, Audio_in_jack2: footprint CONN06_JACK_ACJS_15P75X25_AMP -> audiojack:CONN06_JACK_ACJS_15P75X25_AMP
- I2C_Output_Pins1: footprint Connector_PinSocket_1.27mm:PinSocket_1x02_P1.27mm_Vertical -> Connector_PinHeader_2.54mm:PinHeader_1x02_P2.54mm_Vertical
- J1: footprint Connector_PinHeader_1.00mm:PinHeader_1x02_P1.00mm_Vertical -> Connector_PinSocket_2.54mm:PinSocket_1x02_P2.54mm_Vertical
Changed lines of the file:
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@@
 			)
 		)
-		(property "Footprint" "CONN06_JACK_ACJS_15P75X25_AMP"
+		(property "Footprint" "audiojack:CONN06_JACK_ACJS_15P75X25_AMP"
 			(at 205.74 38.1 0)
 			(effects
@@
 			)
 		)
-		(property "Footprint" "Connector_PinSocket_1.27mm:PinSocket_1x02_P1.27mm_Vertical"
+		(property "Footprint" "Connector_PinHeader_2.54mm:PinHeader_1x02_P2.54mm_Vertical"
 			(at 130.81 104.14 0)
 			(effects
@@
 			)
 		)
-		(property "Footprint" "CONN06_JACK_ACJS_15P75X25_AMP"
+		(property "Footprint" "audiojack:CONN06_JACK_ACJS_15P75X25_AMP"
 			(at 222.25 64.77 0)
 			(effects
@@
 			)
 		)
-		(property "Footprint" "Connector_PinHeader_1.00mm:PinHeader_1x02_P1.00mm_Vertical"
+		(property "Footprint" "Connector_PinSocket_2.54mm:PinSocket_1x02_P2.54mm_Vertical"
 			(at 127 116.84 0)
 			(effects
