File: Daisy_Amps/untitled.kicad_sch (KiCad schematic)
At the start: 0 parts

Commit message: schematic done
Parts:
- added C10, C9: 2.2NF, Capacitor_SMD:C_0805_2012Metric, symbol Device:C
- added C11, C12: 100NF, Capacitor_SMD:C_0805_2012Metric_Pad1.18x1.45mm_HandSolder, symbol Device:C
- added C3, C4, C7, C8: 10UF, Capacitor_SMD:C_0805_2012Metric_Pad1.18x1.45mm_HandSolder, symbol Device:C
- added R10, R12: 100R, Resistor_SMD:R_0805_2012Metric_Pad1.20x1.40mm_HandSolder, symbol Device:R
- added R11, R13, R16, R7, R8, R9: 2M, Resistor_SMD:R_0805_2012Metric_Pad1.20x1.40mm_HandSolder, symbol Device:R
- added R14, R15: 3.3K, Resistor_SMD:R_0805_2012Metric, symbol Device:R
- added U2: OPA2134, Package_DIP:DIP-8_W7.62mm_LongPads, symbol Amplifier_Operational:OPA2134
Connections:
- net Audio_out_daisy_left: now also R14.1
- net Audio_out_daisy_right: now also R15.1
- new net: C4.2, R16.2, R9.1, U2.5 (+)
- new net: R10.1, U2.6 (-), U2.7
- new net: R12.1, U2.1, U2.2 (-)
- new net: C3.2, R7.2, R8.1, U2.3 (+)
- new net: C7.1, R10.2
- new net: C8.1, R12.2
- new net: C4.1, C9.1, R14.2
- new net: C10.1, C3.1, R15.2
- new net +5V: C11.1, C12.1, R16.1, R7.1, U2.8 (V+)
- new net Audio_out_jack_left: C7.2, R11.1
- new net Audio_out_jack_right: C8.2, R13.1
- new net GND: C10.2, C11.2, C12.2, C9.2, R11.2, R13.2, R8.2, R9.2, U2.4 (V-)
Other:
- note added: "Simple RC Low Pass Filter at ~22kHz to remove out of band noise from Seed Rev7"
