File: imu_esp_pcb/imu_esp_pcb.kicad_pcb (KiCad board)
At the start: 2 copper layers, 19 parts, among them J3 Conn_01x02_Pin, U1 MPU-6050, U2 ESP32-C3-WROOM-02, U3 PTS647SM38SMTR2LFS, U4 XC6206P332MR-G, U5 1N5819HW-7-F

Commit message: PCB changes
Parts:
- added R4: 0, Resistor_SMD:R_0805_2012Metric_Pad1.20x1.40mm_HandSolder, F.Cu at (104.5, 87.0)
- added R5: 0, Resistor_SMD:R_0805_2012Metric_Pad1.20x1.40mm_HandSolder, F.Cu at (95.0, 90.5)
- added R6: 0, Resistor_SMD:R_0805_2012Metric_Pad1.20x1.40mm_HandSolder, F.Cu at (94.0, 71.0)
- moved C4 2.00 mm to (92.5, 84.5)
- moved C1 2.00 mm to (95.0, 84.5)
- moved C9 0.96 mm to (98.5, 80.5)
Connections:
- U1 pad 24: SDA -> Net-(U1-SDA)
Routing:
- net GND: track 2.65 -> 36.1 mm
- net SDA: track 14.8 -> 5.22 mm, vias 2 -> 0
- net Net-(U1-SDA): track 0.00 -> 6.98 mm
- net Net-(U4-VIN): track 11.6 -> 9.58 mm
- net Net-(U1-CPOUT): track 10.8 -> 9.54 mm
- net Net-(U1-REGOUT): track 8.42 -> 7.60 mm
- net Net-(U1-VLOGIC): track 8.65 -> 9.17 mm
- net +3.3V: track 90.9 -> 91.3 mm, vias 2 -> 0
- removed copper zone on B.Cu, net GND
Other:
- board outline added: 48.5 x 26 mm
